File: LoRaBoard.sch (KiCad schematic (older format))
At the start: 16 parts

Commit message: PCB layout
Parts:
- removed J?: SPI, symbol CONN_01X04
- removed J?: ADC, symbol CONN_01X07
- removed S?: SWITCH-SPDT-SMD-A, SWITCH-SPST-SMD-A, symbol SWITCH-SPDT-SMD-A
- removed SW?: Boot, BTN_CK_KSS, symbol SWITCH_PUSHBUTTONC&K_KSS
- removed SW?: Reset, BTN_CK_KSS, symbol SWITCH_PUSHBUTTONC&K_KSS
- added D1, D2: LED, LEDs:LED_0603, symbol LED
- added J4: GPIO, Pin_Headers:Pin_Header_Straight_1x04_Pitch2.54mm, symbol CONN_01X04
- added J5: CONN_01X08, Pin_Headers:Pin_Header_Straight_1x08_Pitch2.54mm, symbol CONN_01X08
- added J6: CONN_01X02, Pin_Headers:Pin_Header_Straight_1x02_Pitch2.54mm, symbol CONN_01X02
- added R2, R3: 10k, Resistors_SMD:R_0603, symbol RESISTOR0603-RES
- added S1: SWITCH-SPDTPTH2, SparkFun-Electromechanical:SWITCH-SPST-SMD-A, symbol SWITCH-SPDTPTH2
- added SW1: RESET, adafruit:EVQ-Q2, symbol SPST_TACT-EVQQ2
- C1, C2, C3: renamed from C?; footprint (none) -> Capacitors_SMD:C_0603
- J1, J2, J3: renamed from J?; footprint (none) -> Pin_Headers:Pin_Header_Straight_1x03_Pitch2.54mm
- J7: renamed from J?; footprint (none) -> Pin_Headers:Pin_Header_Straight_1x02_Pitch2.54mm
- R1: renamed from R?; value RESISTOR0603-RES -> 10k; footprint 0603-RES -> Resistors_SMD:R_0603
- U1: renamed from U?; footprint (none) -> im880b:im880b
- U2: renamed from U?; footprint SOT23-5 -> TO_SOT_Packages_SMD:SOT-23-5
- X1: renamed from X?; footprint SMA90_DIP -> adafruit:SMA90_DIP
Connections:
- net labels added: P10, P11, P12, P13, P14, P15, P17, P5, P6, P7, P8, P9
- wire segments 50 -> 104
Other:
- note added: "3mm holes size\n"
- note added: "Indication\n"
- note added: "P1 - SWCLK - PA_14\nP2 - SWDIO - PA_13\n\n"
- note added: "P12 - I2C1_SCL - PB_8\nP13 - I2C1_SDA - PB_9\n"
- note added: "P5 - DIO/UART1_CTS - PA_11\nP6 - DIO/UART1_RTS - PA_12\nP11- DIO - PA_8\n"
- note added: "P7 - ADC_IN20/SPI2_MISO - PB_14 \nP8 - ADC_IN21/SPI2_MOSI - PB_15\nP9 - ADC_IN19/SPI2_CLK - PB_13\nP10 - ADC_IN18/SPI2_NSS - PB_12\nP14 - ADC_IN1 - PA_1 \nP15 - ADC_IN0 - PA_0\nP17 - ADC_IN3 - PA_3\n"
- note added: "TXD - USART1_TXD - PA_9\nRXD - USART1_RXD - PA_10/PB_6"
- moved on the sheet: C1, C2, C3, J1, J2, J3, J7, R1, U1, U2, X1

Commit message: 60% complete
Parts:
- J5: value CONN_01X08 -> ADC/SPI
Connections:
- net GND: now also J4.1 (P1); no longer J4.4 (P4)
- net P11: now also J4.4 (P4); no longer J4.3 (P3)
- net P5: now also J4.3 (P3); no longer J4.1 (P1)
Changed lines of the file:
@@
 P 1050 4550
 F 0 "J5" H 1050 5000 50  0000 C CNN
-F 1 "CONN_01X08" V 1150 4550 50  0000 C CNN
+F 1 "ADC/SPI" V 1150 4550 50  0000 C CNN
 F 2 "Pin_Headers:Pin_Header_Straight_1x08_Pitch2.54mm" H 1050 4550 50  0001 C CNN
 F 3 "" H 1050 4550 50  0001 C CNN
@@
 	950  2200 950  2500
 Text Label 800  2400 2    60   ~ 0
-P5
+GND
 Text Label 950  2500 2    60   ~ 0
 P6
@@
 	7800 1200 7800 1250
 Wire Wire Line
-	1150 2250 1200 2250
-$Comp
-L GND #PWR031
-U 1 1 58D8EB65
-P 1200 2250
-F 0 "#PWR031" H 1200 2000 50  0001 C CNN
-F 1 "GND" H 1200 2100 50  0000 C CNN
-F 2 "" H 1200 2250 50  0001 C CNN
-F 3 "" H 1200 2250 50  0001 C CNN
-	1    1200 2250
-	0    -1   -1   0
-$EndComp
-Wire Wire Line
 	1150 2200 1150 2250
 Text Label 1100 2400 0    60   ~ 0
-P11
+P5
 Wire Wire Line
 	1050 2400 1100 2400
@@
 	10450 4550 10550 4550
 $Comp
-L GND #PWR032
+L GND #PWR031
 U 1 1 58D90E30
 P 10900 4600
-F 0 "#PWR032" H 10900 4350 50  0001 C CNN
+F 0 "#PWR031" H 10900 4350 50  0001 C CNN
 F 1 "GND" H 10900 4450 50  0000 C CNN
 F 2 "" H 10900 4600 50  0001 C CNN
@@
 Text Notes 6850 950  0    60   ~ 0
 Indication\n
+Text Label 1150 2250 0    60   ~ 0
+P11
 $EndSCHEMATC
