File: _saved_LoRaBoard.sch (KiCad schematic (older format))
At the start: 22 parts, among them J1 Prog, J2 I2C, J3 UART, J4 GPIO, J5 ADC/SPI, J6 CONN_01X02, J7 PWR, SW1 SWITCH_PUSHBUTTONC&K_KSS, U1 im880b, U2 LDO-TPS78233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

Commit message: LoRaBoard Done
Parts:
- gave numbers to parts that had none: 2
Changed lines of the file:
@@
 	10350 6000 10350 6100
 $Comp
-L RESISTOR0603-RES R?
+L RESISTOR0603-RES R5
 U 1 1 58E2215E
 P 10750 900
-F 0 "R?" H 10600 959 50  0000 L BNN
+F 0 "R5" H 10600 959 50  0000 L BNN
 F 1 "10k" H 10600 770 50  0000 L BNN
 F 2 "Resistors_SMD:R_0603" H 10780 1050 20  0001 C CNN
@@
 $EndComp
 $Comp
-L RESISTOR0603-RES R?
+L RESISTOR0603-RES R4
 U 1 1 58E22264
 P 10450 650
-F 0 "R?" H 10300 709 50  0000 L BNN
+F 0 "R4" H 10300 709 50  0000 L BNN
 F 1 "33k" H 10300 520 50  0000 L BNN
 F 2 "Resistors_SMD:R_0603" H 10480 800 20  0001 C CNN
@@
 	10750 1100 10750 1150
 $Comp
-L GND #PWR?
+L GND #PWR032
 U 1 1 58E22571
 P 10750 1150
-F 0 "#PWR?" H 10750 900 50  0001 C CNN
+F 0 "#PWR032" H 10750 900 50  0001 C CNN
 F 1 "GND" H 10750 1000 50  0000 C CNN
 F 2 "" H 10750 1150 50  0001 C CNN
@@
 $EndComp
 $Comp
-L +BATT #PWR?
+L +BATT #PWR033
 U 1 1 58E225BE
 P 10200 650
-F 0 "#PWR?" H 10200 500 50  0001 C CNN
+F 0 "#PWR033" H 10200 500 50  0001 C CNN
 F 1 "+BATT" H 10200 790 50  0000 C CNN
 F 2 "" H 10200 650 50  0001 C CNN
