File: LoRaBoard.kicad_pcb (KiCad board)
At the start: 2 copper layers, 20 parts, among them J1 Prog, J2 I2C, J3 UART, J4 GPIO, J5 CONN_01X08, J6 CONN_01X02, J7 PWR, SW1 RESET, U1 im880b, U2 LDO-TPS78233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

Commit message: 60% complete
Parts:
- C2, C3, U2: moved to B.Cu
- J5: value CONN_01X08 -> ADC/SPI
- moved D2 93.5 mm to (159.4, 99.5)
- moved R3 93.1 mm to (159.3, 101.7), turned to 180 degrees
- moved D1 91.0 mm to (154.8, 97.7)
- moved R2 84.4 mm to (154.8, 99.7), turned to 180 degrees
- moved J5 81.4 mm to (134.8, 131.7), turned to 180 degrees
- moved SW1 75.8 mm to (165.8, 116.5), turned to 90 degrees
- moved U2 68.6 mm to (149.8, 107.5), turned to 180 degrees
- moved C1 66.5 mm to (150.1, 131.1)
- moved J6 64.1 mm to (153.2, 134.4), turned to 90 degrees
- moved J3 59.5 mm to (147.9, 134.6), turned to 270 degrees
- moved S1 57.4 mm to (147.8, 96.0)
- moved J7 56.5 mm to (145.1, 101.4), turned to 90 degrees
- moved R1 51.8 mm to (150.9, 100.2), turned to 90 degrees
- moved C3 45.1 mm to (146.1, 107.6), turned to 270 degrees
- moved J4 40.4 mm to (135.1, 109.0), turned to 180 degrees
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Connections:
- J4 pad 1: /P5 -> GND
- J4 pad 3: /P11 -> /P5
- J4 pad 4: GND -> /P11
Routing:
- net /RESET: track 0.00 -> 33.8 mm, vias 0 -> 2
- net /P17: track 0.00 -> 27.6 mm, vias 0 -> 1
- net /P15: track 0.00 -> 25.9 mm, vias 0 -> 1
- net /P14: track 0.00 -> 25.6 mm, vias 0 -> 1
- net /RXD: track 0.00 -> 23.4 mm, vias 0 -> 1
- net /JTMS: track 0.00 -> 20.1 mm, vias 0 -> 1
- net /P6: track 0.00 -> 19.3 mm
- net /P5: track 0.00 -> 19.3 mm
- net /TXD: track 0.00 -> 17.6 mm, vias 0 -> 1
- net /P10: track 0.00 -> 17.3 mm, vias 0 -> 1
- net /JTCK: track 0.00 -> 14.8 mm, vias 0 -> 1
- net +3V3: track 0.00 -> 14.4 mm
- net /P9: track 0.00 -> 14.4 mm, vias 0 -> 1
- net /P7: track 0.00 -> 9.34 mm
- net /P8: track 0.00 -> 7.36 mm, vias 0 -> 1
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- added copper zone on B.Cu, net +3V3
- added copper zone on B.Cu, net +BATT
- added copper zone on B.Cu, net GND

Commit message: LoRaBoard Done
Parts:
- added R4: 33k, Resistors_SMD:R_0603, F.Cu at (153.3, 106.9)
- added R5: 10k, Resistors_SMD:R_0603, F.Cu at (153.3, 108.6)
- added REF**: MountingHole_2.2mm_M2_DIN965, Mounting_Holes:MountingHole_2.2mm_M2_DIN965, F.Cu at (178.9, 100.8)
- added REF**: MountingHole_2.2mm_M2_DIN965, Mounting_Holes:MountingHole_2.2mm_M2_DIN965, F.Cu at (140.8, 135.6)
- added REF**: MountingHole_2.2mm_M2_DIN965, Mounting_Holes:MountingHole_2.2mm_M2_DIN965, F.Cu at (141.0, 100.6)
- R1: moved to B.Cu
- S1: footprint SparkFun-Electromechanical:SWITCH-SPST-SMD-A -> SparkFun-Electromechanical:SWITCH-SPDT-SMD
- SW1: value RESET -> SWITCH_PUSHBUTTONC&K_KSS; footprint adafruit:EVQ-Q2 -> BTN_CK_KSS
- moved J3 28.1 mm to (176.0, 134.0)
- moved J6 26.2 mm to (177.0, 123.6), turned to 0 degrees
- moved S1 19.7 mm to (167.2, 99.2)
- moved J4 19.0 mm to (144.0, 125.7)
- moved C3 12.1 mm to (157.8, 110.8), turned to 0 degrees
- moved J5 11.9 mm to (146.5, 134.0), turned to 90 degrees
- moved J1 10.7 mm to (143.8, 107.1), turned to 0 degrees
- moved J7 10.6 mm to (155.7, 101.4)
- moved D2 10.4 mm to (149.0, 100.0), turned to 180 degrees
- moved R3 10.4 mm to (148.9, 102.2), turned to 0 degrees
- moved SW1 9.95 mm to (175.2, 113.4), turned to 0 degrees
- moved D1 9.34 mm to (145.8, 100.0)
- moved R2 9.31 mm to (145.8, 102.2)
- moved X1 8.61 mm to (174.5, 107.0)
- moved C1 7.95 mm to (158.0, 131.2)
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Connections:
- J5 pad 5: /P14 -> /P17
- J5 pad 7: /P17 -> /P14
Routing:
- net /P11: track 0.40 -> 71.4 mm, vias 0 -> 2
- net +3V3: track 14.4 -> 72.1 mm, vias 0 -> 5
- net /RESET: track 33.8 -> 89.0 mm
- net GND: track 3.52 -> 53.6 mm, vias 0 -> 12
- net /P17: track 27.6 -> 47.2 mm
- net /BOOT: track 0.00 -> 16.9 mm
- net Net-(R1-Pad2): track 0.00 -> 15.5 mm, vias 0 -> 1
- net /P5: track 19.3 -> 5.19 mm
- net /P6: track 19.3 -> 5.41 mm
- net /JTMS: track 20.1 -> 7.22 mm, vias 1 -> 0
- net /P10: track 17.3 -> 5.22 mm, vias 1 -> 0
- net /EN: track 0.00 -> 11.9 mm, vias 0 -> 1
- net /RXD: track 23.4 -> 12.3 mm, vias 1 -> 0
- net /JTCK: track 14.8 -> 4.72 mm, vias 1 -> 0
- net /P9: track 14.4 -> 5.20 mm, vias 1 -> 0
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
Commit message: Done, panelize
Parts:
- removed the REF** at (178.9, 100.8)
- removed the REF** at (140.8, 135.6)
- removed the REF** at (141.0, 100.6)
- added J8: CONN_01X01, Pin_Headers:Pin_Header_Straight_1x01_Pitch2.54mm, F.Cu at (149.6, 101.3)
- added LOGO: , logo:logo, F.Cu at (138.2, 97.7)
- added REF**: MountingHole_2.5mm, Mounting_Holes:MountingHole_2.5mm, F.Cu at (140.8, 132.0)
- added REF**: MountingHole_2.5mm, Mounting_Holes:MountingHole_2.5mm, F.Cu at (174.5, 100.1)
- moved D1 38.4 mm to (170.8, 129.1)
- moved R2 38.0 mm to (170.9, 130.7)
- moved D2 5.14 mm to (144.9, 103.1)
- moved R3 4.09 mm to (144.9, 101.6)
- moved S1 1.94 mm to (165.3, 99.6)
Routing:
- net /P11: track 71.4 -> 57.6 mm
- net +3V3: track 72.1 -> 63.3 mm
- net GND: track 53.6 -> 49.7 mm, vias 12 -> 11
- net Net-(R1-Pad2): track 15.5 -> 12.3 mm
- net /EN: track 11.9 -> 9.92 mm
- net (no net): track 0.87 -> 0.00 mm
- net Net-(D2-Pad2): track 2.20 -> 1.52 mm
- net Net-(D1-Pad2): track 2.22 -> 1.62 mm
Other:
- board outline added: 42 x 41 mm
- board text added: "+"
- board text added: "-"
- board text added: "LoRa DevBoard"

Commit message: Panel added
Parts:
- moved LOGO 4.85 mm to (138.1, 102.5)
- moved J6 0.25 mm to (176.8, 123.6)
Other:
- outline, holes or cut-outs redrawn
Changed lines of the file:
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@@
 (kicad_pcb (version 4) (host pcbnew 4.0.6-e0-6349~53~ubuntu14.04.1)
   (general
-    (links 0)
+    (links 63)
     (no_connects 1)
     (area 128.650001 95.587459 185.850601 142.700001)
     (thickness 1.6)
-    (drawings 9)
-    (tracks 254)
+    (drawings 11)
+    (tracks 255)
     (zones 0)
     (modules 26)
@@
   (page A4)
   (layers
-    (0 F.Cu signal hide)
+    (0 F.Cu signal)
     (31 B.Cu signal)
     (32 B.Adhes user)
@@
   )
   (setup
-    (last_trace_width 0.25)
+    (last_trace_width 0.55)
     (user_trace_width 0.4)
     (user_trace_width 0.45)
@@
     (pad_to_mask_clearance 0)
     (aux_axis_origin 141.8 102)
+    (grid_origin 180 97)
     (visible_elements FFFEFF7F)
     (pcbplotparams
@@
   )
   (module Mounting_Holes:MountingHole_2.5mm (layer F.Cu)
+    (at 174.5 100.1)
+    (descr "Mounting Hole 2.5mm, no annular")
+    (tags "mounting hole 2.5mm no annular")
+    (fp_text reference REF** (at 0 -3.5) (layer F.SilkS) hide
+      (effects (font (size 1 1) (thickness 0.15)))
+    )
+    (fp_text value MountingHole_2.5mm (at 0 3.5) (layer F.Fab)
+      (effects (font (size 1 1) (thickness 0.15)))
+    )
+    (fp_circle (center 0 0) (end 2.5 0) (layer Cmts.User) (width 0.15))
+    (fp_circle (center 0 0) (end 2.75 0) (layer F.CrtYd) (width 0.05))
+    (pad 1 np_thru_hole circle (at 0 0) (size 2.5 2.5) (drill 2.5) (layers *.Cu *.Mask))
+  )
+  (module Mounting_Holes:MountingHole_2.5mm (layer F.Cu)
     (at 140.8 132)
     (descr "Mounting Hole 2.5mm, no annular")
@@
   )
   (module Pin_Headers:Pin_Header_Straight_1x02_Pitch2.54mm (layer F.Cu)
-    (at 177 123.6)
+    (at 176.75 123.6)
     (descr "Through hole straight pin header, 1x02, 2.54mm pitch, single row")
     (tags "Through hole pin header THT 1x02 2.54mm single row")
@@
     (tags "resistor 0603")
     (attr smd)
-    (fp_text reference R3 (at 0 -1.45) (layer F.SilkS)
+    (fp_text reference R3 (at 1.55 -1.15) (layer F.SilkS)
       (effects (font (size 1 1) (thickness 0.15)))
     )
@@
     )
   )
-  (module Mounting_Holes:MountingHole_2.5mm (layer F.Cu)
-    (at 174.5 100.1)
-    (descr "Mounting Hole 2.5mm, no annular")
-    (tags "mounting hole 2.5mm no annular")
-    (fp_text reference REF** (at 0 -3.5) (layer F.SilkS) hide
-      (effects (font (size 1 1) (thickness 0.15)))
-    )
-    (fp_text value MountingHole_2.5mm (at 0 3.5) (layer F.Fab)
-      (effects (font (size 1 1) (thickness 0.15)))
-    )
-    (fp_circle (center 0 0) (end 2.5 0) (layer Cmts.User) (width 0.15))
-    (fp_circle (center 0 0) (end 2.75 0) (layer F.CrtYd) (width 0.05))
-    (pad 1 np_thru_hole circle (at 0 0) (size 2.5 2.5) (drill 2.5) (layers *.Cu *.Mask))
-  )
   (module logo:logo (layer F.Cu)
-    (at 138.2 97.65)
+    (at 138.1 102.5)
     (fp_text reference LOGO (at 0 5) (layer F.SilkS) hide
       (effects (font (thickness 0.3)))
@@
       (xy 2.975 5.45)) (layer F.SilkS) (width 0.01))
   )
+  (gr_line (start 178.47 97) (end 141 97) (angle 90) (layer Edge.Cuts) (width 0.1))
+  (gr_line (start 180 136.49) (end 180 98.49) (angle 90) (layer Edge.Cuts) (width 0.1))
+  (gr_line (start 139.55 138) (end 178.46 138) (angle 90) (layer Edge.Cuts) (width 0.1))
+  (gr_line (start 138 100.01) (end 138 136.54) (angle 90) (layer Edge.Cuts) (width 0.1))
+  (gr_arc (start 178.5 98.5) (end 178.5 97) (angle 90) (layer Edge.Cuts) (width 0.1))
+  (gr_arc (start 178.5 136.5) (end 180 136.5) (angle 90) (layer Edge.Cuts) (width 0.1))
+  (gr_arc (start 139.5 136.5) (end 139.5 138) (angle 90) (layer Edge.Cuts) (width 0.1))
+  (gr_arc (start 141 100) (end 138 100) (angle 90) (layer Edge.Cuts) (width 0.1))
   (gr_text + (at 174.1 129) (layer F.SilkS)
     (effects (font (size 1.5 1.5) (thickness 0.3)))
@@
     (effects (font (size 1.5 1.5) (thickness 0.3)))
   )
-  (gr_line (start 138 97) (end 138 138) (layer Edge.Cuts) (width 0.1))
-  (gr_line (start 180 97) (end 138 97) (layer Edge.Cuts) (width 0.1))
-  (gr_line (start 180 137.95) (end 180 97) (layer Edge.Cuts) (width 0.1))
-  (gr_line (start 138 138) (end 180 137.95) (layer Edge.Cuts) (width 0.1))
-  (gr_text "LoRa DevBoard\n" (at 139.4 111.85 90) (layer F.SilkS)
+  (gr_text "LoRa DevBoard\n" (at 139.65 117.35 90) (layer F.SilkS)
     (effects (font (size 1.5 1.5) (thickness 0.3)))
   )
-  (dimension 41 (width 0.3) (layer Dwgs.User)
-    (gr_text "41.000 mm" (at 135.15 117.5 90) (layer Dwgs.User)
-      (effects (font (size 1.5 1.5) (thickness 0.3)))
-    )
-    (feature1 (pts (xy 138 97) (xy 133.8 97)))
-    (feature2 (pts (xy 138 138) (xy 133.8 138)))
-    (crossbar (pts (xy 136.5 138) (xy 136.5 97)))
-    (arrow1a (pts (xy 136.5 97) (xy 137.086421 98.126504)))
-    (arrow1b (pts (xy 136.5 97) (xy 135.913579 98.126504)))
-    (arrow2a (pts (xy 136.5 138) (xy 137.086421 136.873496)))
-    (arrow2b (pts (xy 136.5 138) (xy 135.913579 136.873496)))
-  )
-  (dimension 42 (width 0.3) (layer Dwgs.User)
-    (gr_text "42.000 mm" (at 159 141.35) (layer Dwgs.User)
-      (effects (font (size 1.5 1.5) (thickness 0.3)))
-    )
-    (feature1 (pts (xy 180 138) (xy 180 142.7)))
-    (feature2 (pts (xy 138 138) (xy 138 142.7)))
-    (crossbar (pts (xy 138 140) (xy 180 140)))
-    (arrow1a (pts (xy 180 140) (xy 178.873496 140.586421)))
-    (arrow1b (pts (xy 180 140) (xy 178.873496 139.413579)))
-    (arrow2a (pts (xy 138 140) (xy 139.126504 140.586421)))
-    (arrow2b (pts (xy 138 140) (xy 139.126504 139.413579)))
-  )
+  (segment (start 176.75 123.6) (end 176.75 122.2) (width 0.55) (layer F.Cu) (net 1))
+  (segment (start 176.75 122.2) (end 177 121.95) (width 0.55) (layer F.Cu) (net 1))
+  (segment (start 177 121.95) (end 177 119.3975) (width 0.55) (layer F.Cu) (net 1))
   (via (at 148.8 103.6) (size 0.6) (drill 0.4) (layers F.Cu B.Cu) (net 1))
   (segment (start 146.5 101.6) (end 147.7 102.8) (width 0.6) (layer F.Cu) (net 1))
@@
   (segment (start 170.2 114.00143) (end 170.80143 113.4) (width 0.6) (layer F.Cu) (net 1))
   (segment (start 170.80143 113.4) (end 172.25106 113.4) (width 0.6) (layer F.Cu) (net 1) (status 20))
-  (segment (start 177 123.6) (end 177 119.3975) (width 0.6) (layer F.Cu) (net 1) (status 10))
   (segment (start 154.8 111.8) (end 154.8 111) (width 1) (layer B.Cu) (net 1))
   (segment (start 154.8 123.2) (end 154.8 111.8) (width 1) (layer F.Cu) (net 1))
@@
   (via (at 170.2 115.6) (size 0.6) (drill 0.4) (layers F.Cu B.Cu) (net 1))
   (segment (start 171.85148 116.59954) (end 171.85148 116.45148) (width 0.6) (layer F.Cu) (net 1))
-  (segment (start 176.8 123.4) (end 177 123.6) (width 0.6) (layer F.Cu) (net 1) (status 30))
   (segment (start 171.85148 117.74898) (end 171.85148 116.59954) (width 0.55) (layer F.Cu) (net 1))
   (segment (start 158.75 131.25) (end 159.35 131.25) (width 0.55) (layer F.Cu) (net 1) (status 10))
@@
   (segment (start 156.66 134) (end 156.66 128.34) (width 0.6) (layer B.Cu) (net 21) (status 10))
   (segment (start 167.5347 111.2) (end 167.8311 110.9036) (width 0.6) (layer F.Cu) (net 21) (status 30))
-  (segment (start 167.8311 116.9036) (end 168.7036 116.9036) (width 0.55) (layer F.Cu) (net 22) (status 30))
-  (segment (start 174 119.4) (end 174.8 120.2) (width 0.55) (layer F.Cu) (net 22))
-  (segment (start 168.7036 116.9036) (end 169.777549 117.977549) (width 0.55) (layer F.Cu) (net 22) (status 10))
-  (segment (start 169.777549 119.177549) (end 170 119.4) (width 0.55) (layer F.Cu) (net 22))
-  (segment (start 174.8 120.2) (end 174.8 125.6) (width 0.55) (layer F.Cu) (net 22))
+  (segment (start 167.8311 116.9036) (end 168.7036 116.9036) (width 0.55) (layer F.Cu) (net 22))
+  (segment (start 174.8 125.7) (end 175.24 126.14) (width 0.55) (layer F.Cu) (net 22))
+  (segment (start 168.7036 116.9036) (end 169.777549 117.977549) (width 0.55) (layer F.Cu) (net 22))
   (segment (start 169.777549 117.977549) (end 169.777549 119.177549) (width 0.55) (layer F.Cu) (net 22))
-  (segment (start 174.8 125.6) (end 175.34 126.14) (width 0.55) (layer F.Cu) (net 22))
+  (segment (start 169.777549 119.177549) (end 170 119.4) (width 0.55) (layer F.Cu) (net 22))
+  (segment (start 175.24 126.14) (end 176.75 126.14) (width 0.55) (layer F.Cu) (net 22))
   (segment (start 170 119.4) (end 174 119.4) (width 0.55) (layer F.Cu) (net 22))
-  (segment (start 175.34 126.14) (end 177 126.14) (width 0.55) (layer F.Cu) (net 22) (status 20))
+  (segment (start 174 119.4) (end 174.8 120.2) (width 0.55) (layer F.Cu) (net 22))
+  (segment (start 174.8 120.2) (end 174.8 125.7) (width 0.55) (layer F.Cu) (net 22))
   (segment (start 152.45 105.4) (end 152.45 104.15) (width 0.6) (layer B.Cu) (net 23))
   (segment (start 161.44892 103.7) (end 162.80064 102.34828) (width 0.6) (layer F.Cu) (net 23))

Commit message: PCB complete, panel complete
Parts:
- removed J8: CONN_01X01, Pin_Headers:Pin_Header_Straight_1x01_Pitch2.54mm
- removed the REF** at (174.5, 100.1)
- removed the REF** at (140.8, 132.0)
- removed S1: SWITCH-SPDTPTH2, SparkFun-Electromechanical:SWITCH-SPDT-SMD
- removed SW1: SWITCH_PUSHBUTTONC&K_KSS, BTN_CK_KSS
- removed X1: SMACONNECTOR, adafruit:SMA90_DIP
- added REF**: MountingHole_2.5mm, Mounting_Holes:MountingHole_2.5mm, F.Cu at (127.8, 82.0)
- added REF**: MountingHole_2.5mm, Mounting_Holes:MountingHole_2.5mm, F.Cu at (157.8, 117.2)
- C2, C3: value 0.1u -> 1u
- J1: value Prog -> CONN_01X12; footprint Pin_Headers:Pin_Header_Straight_1x03_Pitch2.54mm -> Pin_Headers:Pin_Header_Straight_1x12_Pitch2.54mm
- J2: value I2C -> CONN_01X08; footprint Pin_Headers:Pin_Header_Straight_1x03_Pitch2.54mm -> Pin_Headers:Pin_Header_Straight_1x08_Pitch2.54mm
- J3: value UART -> CONN_01X09; footprint Pin_Headers:Pin_Header_Straight_1x03_Pitch2.54mm -> Pin_Headers:Pin_Header_Straight_1x09_Pitch2.54mm
- J4: value GPIO -> CONN_COAXIAL; footprint Pin_Headers:Pin_Header_Straight_1x04_Pitch2.54mm -> Connectors:SMA_THT_Jack_Straight
- J5: value ADC/SPI -> SwitchSPST; footprint Pin_Headers:Pin_Header_Straight_1x08_Pitch2.54mm -> Buttons_Switches_SMD:SW_SPST_EVQPE1
- J6: value CONN_01X02 -> CONN_01X01; footprint Pin_Headers:Pin_Header_Straight_1x02_Pitch2.54mm -> Pin_Headers:Pin_Header_Straight_1x01_Pitch2.54mm
- R3, R4, R5: moved to B.Cu
- moved J2 43.2 mm to (130.6, 115.6), turned to 90 degrees
- moved J4 39.3 mm to (155.4, 88.1), turned to 0 degrees
- moved J6 36.4 mm to (140.8, 118.2)
- moved R5 32.6 mm to (130.8, 85.0), turned to 180 degrees
- moved J1 32.1 mm to (122.9, 82.7)
- moved R2 29.9 mm to (148.2, 111.2)
- moved J3 29.6 mm to (153.5, 114.8), turned to 180 degrees
- moved R4 29.4 mm to (133.8, 85.0)
- moved J5 28.6 mm to (124.4, 115.8), turned to 180 degrees
- moved U2 27.5 mm to (138.6, 87.7)
- moved C3 27.5 mm to (138.5, 91.1)
- moved U1 27.5 mm to (128.5, 86.2)
- moved C1 27.3 mm to (138.0, 112.6)
- moved C2 26.9 mm to (138.5, 84.9)
- moved D1 26.9 mm to (149.5, 112.8), turned to 180 degrees
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Connections:
- net /JTMS renamed /3
- J1 pad 1: /JTCK -> /1
- J1 pad 2: GND -> /2
- J2 pad 1: /P12 -> /13
- J2 pad 2: GND -> /14
- J2 pad 3: /P13 -> /15
- J3 pad 1: /TXD -> /21
- J3 pad 3: /RXD -> /23
- J4 pad 1: GND -> /RF
- J4 pad 2: /P6 -> GND
- J5 pad 1: /P7 -> +3V3
- J5 pad 2: /P8 -> /7
- R1 pad 1: +BATT -> Net-(R1-Pad1)
- R1 pad 2: Net-(R1-Pad2) -> +BATT
- R2 pad 2: /P11 -> /20
- R4 pad 1: /P17 -> /29
- R5 pad 1: /P17 -> /29
- U1 pad 1: GND -> /1
- U1 pad 12: /P7 -> /12
- U1 pad 13: /P8 -> /13
- U1 pad 14: /P9 -> /14
- U1 pad 15: /P10 -> /15
- U1 pad 18: /RXD -> /18
- U1 pad 19: /TXD -> /19
- U1 pad 2: /JTCK -> /2
- U1 pad 20: /P11 -> /20
- U1 pad 21: /P12 -> /21
- U1 pad 23: /P13 -> /23
- U1 pad 24: /P14 -> /24
- U1 pad 25: /P15 -> /25
- U1 pad 26: /BOOT -> /26
- U1 pad 29: /P17 -> /29
- U1 pad 4: (no net) -> /4
- U1 pad 5: (no net) -> /5
- U1 pad 7: /RESET -> /7
- U1 pad 8: /P5 -> /8
- U1 pad 9: /P6 -> /9
- U2 pad 3: /EN -> Net-(R1-Pad1)
Routing:
- net /RESET: track 89.0 -> 0.00 mm, vias 2 -> 0
- net /P11: track 57.6 -> 0.00 mm, vias 2 -> 0
- net /P17: track 47.0 -> 0.00 mm, vias 1 -> 0
- net /29: track 0.00 -> 28.8 mm, vias 0 -> 1
- net /7: track 0.00 -> 25.3 mm
- net /P15: track 20.6 -> 0.00 mm, vias 1 -> 0
- net /P14: track 17.4 -> 0.00 mm, vias 1 -> 0
- net /BOOT: track 16.7 -> 0.00 mm
- net /TXD: track 15.7 -> 0.00 mm
- net Net-(R1-Pad2): track 12.3 -> 0.00 mm, vias 1 -> 0
- net /RXD: track 12.3 -> 0.00 mm
- net /21: track 0.00 -> 10.9 mm
- net /EN: track 9.92 -> 0.00 mm, vias 1 -> 0
- net /23: track 0.00 -> 9.50 mm
- net /20: track 0.00 -> 8.75 mm
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- added copper zone on F.Cu, net GND
Other:
- board size 42 x 41 mm -> 40.8 x 42 mm
- net class Default: via_dia 0.6 -> 0.8
- board text added: "LoRa DevBoard v1"
- board text removed: "+"
- board text removed: "-"
- board text removed: "LoRa DevBoard"
